Commit message: traj_opt init

File: src/sim_env/urdf/turtlebot3_burger/common_properties.xacro (robot description, xacro)
@@ -1,33 +1,34 @@
-<?xml version="1.0"?>
+<?xml version="1.0" ?>
 <robot name="xacro_properties" xmlns:xacro="http://ros.org/wiki/xacro">
+  <!-- Init colour -->
   <material name="black">
-    <color rgba="0.0 0.0 0.0 1.0" />
+      <color rgba="0.0 0.0 0.0 1.0"/>
   </material>
   <material name="dark">
-    <color rgba="0.3 0.3 0.3 1.0" />
+    <color rgba="0.3 0.3 0.3 1.0"/>
   </material>
   <material name="light_black">
-    <color rgba="0.4 0.4 0.4 1.0" />
+    <color rgba="0.4 0.4 0.4 1.0"/>
   </material>
   <material name="blue">
-    <color rgba="0.0 0.0 0.8 1.0" />
+    <color rgba="0.0 0.0 0.8 1.0"/>
   </material>
   <material name="green">
-    <color rgba="0.0 0.8 0.0 1.0" />
+    <color rgba="0.0 0.8 0.0 1.0"/>
   </material>
   <material name="grey">
-    <color rgba="0.5 0.5 0.5 1.0" />
+    <color rgba="0.5 0.5 0.5 1.0"/>
   </material>
   <material name="orange">
-    <color rgba="${255/255} ${108/255} ${10/255} 1.0" />
+    <color rgba="${255/255} ${108/255} ${10/255} 1.0"/>
   </material>
   <material name="brown">
-    <color rgba="${222/255} ${207/255} ${195/255} 1.0" />
+    <color rgba="${222/255} ${207/255} ${195/255} 1.0"/>
   </material>
   <material name="red">
-    <color rgba="0.8 0.0 0.0 1.0" />
+    <color rgba="0.8 0.0 0.0 1.0"/>
   </material>
   <material name="white">
-    <color rgba="1.0 1.0 1.0 1.0" />
+    <color rgba="1.0 1.0 1.0 1.0"/>
   </material>
 </robot>

File: src/sim_env/urdf/turtlebot3_burger/turtlebot3_burger.gazebo.xacro (robot description, xacro)
@@ -1,6 +1,6 @@
 <?xml version="1.0"?>
 <robot name="turtlebot3_burger_sim" xmlns:xacro="http://ros.org/wiki/xacro">
-  <xacro:arg name="laser_visual" default="false" />
-  <xacro:arg name="imu_visual" default="false" />
+  <xacro:arg name="laser_visual" default="false"/>
+  <xacro:arg name="imu_visual"   default="false"/>
   <gazebo reference="base_link">
     <material>Gazebo/DarkGrey</material>

File: src/sim_env/urdf/turtlebot3_burger/turtlebot3_burger.urdf.xacro (robot description, xacro)
@@ -1,50 +1,50 @@
-<?xml version="1.0"?>
+<?xml version="1.0" ?>
 <robot name="turtlebot3_burger" xmlns:xacro="http://ros.org/wiki/xacro">
-  <link name="base_footprint" />
+  <link name="base_footprint"/>
   <joint name="base_joint" type="fixed">
-    <parent link="base_footprint" />
-    <child link="base_link" />
-    <origin xyz="0.0 0.0 0.010" rpy="0 0 0" />
+    <parent link="base_footprint"/>
+    <child link="base_link"/>
+    <origin xyz="0.0 0.0 0.010" rpy="0 0 0"/>
   </joint>
   <link name="base_link">
     <visual>
-      <origin xyz="-0.032 0 0.0" rpy="0 0 0" />
+      <origin xyz="-0.032 0 0.0" rpy="0 0 0"/>
       <geometry>
-        <mesh filename="package://sim_env/meshes/turtlebot3/bases/burger_base.stl" scale="0.001 0.001 0.001" />
+        <mesh filename="package://sim_env/meshes/turtlebot3/bases/burger_base.stl" scale="0.001 0.001 0.001"/>
       </geometry>
-      <material name="light_black" />
+      <material name="light_black"/>
     </visual>
     <collision>
-      <origin xyz="-0.032 0 0.070" rpy="0 0 0" />
+      <origin xyz="-0.032 0 0.070" rpy="0 0 0"/>
       <geometry>
-        <box size="0.140 0.140 0.143" />
+        <box size="0.140 0.140 0.143"/>
       </geometry>
     </collision>
     <inertial>
-      <origin xyz="0 0 0" rpy="0 0 0" />
-      <mass value="8.2573504e-01" />
+      <origin xyz="0 0 0" rpy="0 0 0"/>
+      <mass value="8.2573504e-01"/>
       <inertia ixx="2.2124416e-03" ixy="-1.2294101e-05" ixz="3.4938785e-05"
-        iyy="2.1193702e-03" iyz="-5.0120904e-06"
-        izz="2.0064271e-03" />
+               iyy="2.1193702e-03" iyz="-5.0120904e-06"
+               izz="2.0064271e-03" />
     </inertial>
   </link>
   <joint name="wheel_left_joint" type="continuous">
-    <parent link="base_link" />
-    <child link="wheel_left_link" />
-    <origin xyz="0.0 0.08 0.023" rpy="-1.57 0 0" />
-    <axis xyz="0 0 1" />
+    <parent link="base_link"/>
+    <child link="wheel_left_link"/>
+    <origin xyz="0.0 0.08 0.023" rpy="-1.57 0 0"/>
+    <axis xyz="0 0 1"/>
   </joint>
   <link name="wheel_left_link">
     <visual>
-      <origin xyz="0 0 0" rpy="1.57 0 0" />
+      <origin xyz="0 0 0" rpy="1.57 0 0"/>
       <geometry>
-        <mesh filename="package://sim_env/meshes/turtlebot3/wheels/left_tire.stl" scale="0.001 0.001 0.001" />
+        <mesh filename="package://sim_env/meshes/turtlebot3/wheels/left_tire.stl" scale="0.001 0.001 0.001"/>
       </geometry>
-      <material name="dark" />
+      <material name="dark"/>
     </visual>
     <collision>
-      <origin xyz="0 0 0" rpy="0 0 0" />
+      <origin xyz="0 0 0" rpy="0 0 0"/>
       <geometry>
-        <cylinder length="0.018" radius="0.033" />
+        <cylinder length="0.018" radius="0.033"/>
       </geometry>
     </collision>
@@ -53,26 +53,26 @@
       <mass value="2.8498940e-02" />
       <inertia ixx="1.1175580e-05" ixy="-4.2369783e-11" ixz="-5.9381719e-09"
-        iyy="1.1192413e-05" iyz="-1.4400107e-11"
-        izz="2.0712558e-05" />
-    </inertial>
+               iyy="1.1192413e-05" iyz="-1.4400107e-11"
+               izz="2.0712558e-05" />
+      </inertial>
   </link>
   <joint name="wheel_right_joint" type="continuous">
-    <parent link="base_link" />
-    <child link="wheel_right_link" />
-    <origin xyz="0.0 -0.080 0.023" rpy="-1.57 0 0" />
-    <axis xyz="0 0 1" />
+    <parent link="base_link"/>
+    <child link="wheel_right_link"/>
+    <origin xyz="0.0 -0.080 0.023" rpy="-1.57 0 0"/>
+    <axis xyz="0 0 1"/>
   </joint>
   <link name="wheel_right_link">
     <visual>
-      <origin xyz="0 0 0" rpy="1.57 0 0" />
+      <origin xyz="0 0 0" rpy="1.57 0 0"/>
       <geometry>
-        <mesh filename="package://sim_env/meshes/turtlebot3/wheels/right_tire.stl" scale="0.001 0.001 0.001" />
+        <mesh filename="package://sim_env/meshes/turtlebot3/wheels/right_tire.stl" scale="0.001 0.001 0.001"/>
       </geometry>
-      <material name="dark" />
+      <material name="dark"/>
     </visual>
     <collision>
-      <origin xyz="0 0 0" rpy="0 0 0" />
+      <origin xyz="0 0 0" rpy="0 0 0"/>
       <geometry>
-        <cylinder length="0.018" radius="0.033" />
+        <cylinder length="0.018" radius="0.033"/>
       </geometry>
     </collision>
@@ -81,18 +81,18 @@
       <mass value="2.8498940e-02" />
       <inertia ixx="1.1175580e-05" ixy="-4.2369783e-11" ixz="-5.9381719e-09"
-        iyy="1.1192413e-05" iyz="-1.4400107e-11"
-        izz="2.0712558e-05" />
-    </inertial>
+               iyy="1.1192413e-05" iyz="-1.4400107e-11"
+               izz="2.0712558e-05" />
+      </inertial>
   </link>
   <joint name="caster_back_joint" type="fixed">
-    <parent link="base_link" />
-    <child link="caster_back_link" />
-    <origin xyz="-0.081 0 -0.004" rpy="-1.57 0 0" />
+    <parent link="base_link"/>
+    <child link="caster_back_link"/>
+    <origin xyz="-0.081 0 -0.004" rpy="-1.57 0 0"/>
   </joint>
   <link name="caster_back_link">
     <collision>
-      <origin xyz="0 0.001 0" rpy="0 0 0" />
+      <origin xyz="0 0.001 0" rpy="0 0 0"/>
       <geometry>
-        <box size="0.030 0.009 0.020" />
+        <box size="0.030 0.009 0.020"/>
       </geometry>
     </collision>
@@ -101,31 +101,31 @@
       <mass value="0.005" />
       <inertia ixx="0.001" ixy="0.0" ixz="0.0"
-        iyy="0.001" iyz="0.0"
-        izz="0.001" />
+               iyy="0.001" iyz="0.0"
+               izz="0.001" />
     </inertial>
   </link>
   <joint name="imu_joint" type="fixed">
-    <parent link="base_link" />
-    <child link="imu_link" />
-    <origin xyz="-0.032 0 0.068" rpy="0 0 0" />
+    <parent link="base_link"/>
+    <child link="imu_link"/>
+    <origin xyz="-0.032 0 0.068" rpy="0 0 0"/>
   </joint>
-  <link name="imu_link" />
+  <link name="imu_link"/>
   <joint name="scan_joint" type="fixed">
-    <parent link="base_link" />
-    <child link="base_scan" />
-    <origin xyz="-0.032 0 0.172" rpy="0 0 0" />
+    <parent link="base_link"/>
+    <child link="base_scan"/>
+    <origin xyz="-0.032 0 0.172" rpy="0 0 0"/>
   </joint>
   <link name="base_scan">
     <visual>
-      <origin xyz="0 0 0.0" rpy="0 0 0" />
+      <origin xyz="0 0 0.0" rpy="0 0 0"/>
       <geometry>
-        <mesh filename="package://sim_env/meshes/turtlebot3/sensors/lds.stl" scale="0.001 0.001 0.001" />
+        <mesh filename="package://sim_env/meshes/turtlebot3/sensors/lds.stl" scale="0.001 0.001 0.001"/>
       </geometry>
-      <material name="dark" />
+      <material name="dark"/>
     </visual>
     <collision>
-      <origin xyz="0.015 0 -0.0065" rpy="0 0 0" />
+      <origin xyz="0.015 0 -0.0065" rpy="0 0 0"/>
       <geometry>
-        <cylinder length="0.0315" radius="0.055" />
+        <cylinder length="0.0315" radius="0.055"/>
       </geometry>
     </collision>
@@ -134,6 +134,6 @@
       <origin xyz="0 0 0" />
       <inertia ixx="0.001" ixy="0.0" ixz="0.0"
-        iyy="0.001" iyz="0.0"
-        izz="0.001" />
+               iyy="0.001" iyz="0.0"
+               izz="0.001" />
     </inertial>
   </link>

File: src/sim_env/urdf/turtlebot3_burger/turtlebot3_burger.xacro (robot description, xacro)
@@ -1,6 +1,6 @@
-<?xml version="1.0"?>
+<?xml version="1.0" ?>
 <robot name="turtlebot3_burger" xmlns:xacro="http://ros.org/wiki/xacro">
-  <xacro:include filename="$(find sim_env)/urdf/turtlebot3_burger/common_properties.xacro" />
-  <xacro:include filename="$(find sim_env)/urdf/turtlebot3_burger/turtlebot3_burger.gazebo.xacro" />
-  <xacro:include filename="$(find sim_env)/urdf/turtlebot3_burger/turtlebot3_burger.urdf.xacro" />
+  <xacro:include filename="$(find sim_env)/urdf/turtlebot3_burger/common_properties.xacro"/>
+  <xacro:include filename="$(find sim_env)/urdf/turtlebot3_burger/turtlebot3_burger.gazebo.xacro"/>
+  <xacro:include filename="$(find sim_env)/urdf/turtlebot3_burger/turtlebot3_burger.urdf.xacro"/>
 </robot>

File: src/sim_env/urdf/turtlebot3_waffle/turtlebot3_waffle.gazebo.xacro (robot description, xacro)
@@ -1,7 +1,7 @@
 <?xml version="1.0"?>
 <robot name="turtlebot3_waffle_sim" xmlns:xacro="http://ros.org/wiki/xacro">
-  <xacro:arg name="laser_visual" default="false" />
-  <xacro:arg name="camera_visual" default="false" />
-  <xacro:arg name="imu_visual" default="false" />
+  <xacro:arg name="laser_visual"  default="false"/>
+  <xacro:arg name="camera_visual" default="false"/>
+  <xacro:arg name="imu_visual"    default="false"/>
   <gazebo reference="base_link">
     <material>Gazebo/DarkGrey</material>
@@ -139,15 +139,15 @@
       <visualize>$(arg camera_visual)</visualize>
       <camera>
-        <horizontal_fov>1.3439</horizontal_fov>
-        <image>
-          <width>1920</width>
-          <height>1080</height>
-          <format>R8G8B8</format>
-        </image>
-        <depth_camera></depth_camera>
-        <clip>
-          <near>0.03</near>
-          <far>100</far>
-        </clip>
+          <horizontal_fov>1.3439</horizontal_fov>
+          <image>
+              <width>1920</width>
+              <height>1080</height>
+              <format>R8G8B8</format>
+          </image>
+          <depth_camera></depth_camera>
+          <clip>
+              <near>0.03</near>
+              <far>100</far>
+          </clip>
       </camera>
       <plugin name="camera_controller" filename="libgazebo_ros_openni_kinect.so">
@@ -163,10 +163,10 @@
         <depthImageCameraInfoTopicName>depth/camera_info</depthImageCameraInfoTopicName>
         <pointCloudCutoff>0.4</pointCloudCutoff>
-        <hackBaseline>0.07</hackBaseline>
-        <distortionK1>0.0</distortionK1>
-        <distortionK2>0.0</distortionK2>
-        <distortionK3>0.0</distortionK3>
-        <distortionT1>0.0</distortionT1>
-        <distortionT2>0.0</distortionT2>
+            <hackBaseline>0.07</hackBaseline>
+            <distortionK1>0.0</distortionK1>
+            <distortionK2>0.0</distortionK2>
+            <distortionK3>0.0</distortionK3>
+            <distortionT1>0.0</distortionT1>
+            <distortionT2>0.0</distortionT2>
         <CxPrime>0.0</CxPrime>
         <Cx>0.0</Cx>
