Commit message: traj_opt init

File: src/sim_env/urdf/turtlebot3_waffle/turtlebot3_waffle.urdf.xacro (robot description, xacro)
@@ -1,54 +1,54 @@
-<?xml version="1.0"?>
+<?xml version="1.0" ?>
 <robot name="turtlebot3_waffle" xmlns:xacro="http://ros.org/wiki/xacro">
-  <xacro:property name="r200_cam_rgb_px" value="0.005" />
-  <xacro:property name="r200_cam_rgb_py" value="0.018" />
-  <xacro:property name="r200_cam_rgb_pz" value="0.013" />
-  <xacro:property name="r200_cam_depth_offset" value="0.01" />
-  <link name="base_footprint" />
+  <xacro:property name="r200_cam_rgb_px" value="0.005"/>
+  <xacro:property name="r200_cam_rgb_py" value="0.018"/>
+  <xacro:property name="r200_cam_rgb_pz" value="0.013"/>
+  <xacro:property name="r200_cam_depth_offset" value="0.01"/>
+  <link name="base_footprint"/>
   <joint name="base_joint" type="fixed">
-    <parent link="base_footprint" />
+    <parent link="base_footprint"/>
     <child link="base_link" />
-    <origin xyz="0 0 0.010" rpy="0 0 0" />
+    <origin xyz="0 0 0.010" rpy="0 0 0"/>
   </joint>
   <link name="base_link">
     <visual>
-      <origin xyz="-0.064 0 0.0" rpy="0 0 0" />
-      <geometry>
-        <mesh filename="package://sim_env/meshes/turtlebot3/bases/waffle_base.stl" scale="0.001 0.001 0.001" />
-      </geometry>
-      <material name="light_black" />
-    </visual>
-    <collision>
-      <origin xyz="-0.064 0 0.047" rpy="0 0 0" />
-      <geometry>
-        <box size="0.266 0.266 0.094" />
-      </geometry>
-    </collision>
-    <inertial>
-      <origin xyz="0 0 0" rpy="0 0 0" />
-      <mass value="1.3729096e+00" />
+      <origin xyz="-0.064 0 0.0" rpy="0 0 0"/>
+      <geometry>
+        <mesh filename="package://sim_env/meshes/turtlebot3/bases/waffle_base.stl" scale="0.001 0.001 0.001"/>
+      </geometry>
+      <material name="light_black"/>
+    </visual>
+    <collision>
+      <origin xyz="-0.064 0 0.047" rpy="0 0 0"/>
+      <geometry>
+        <box size="0.266 0.266 0.094"/>
+      </geometry>
+    </collision>
+    <inertial>
+      <origin xyz="0 0 0" rpy="0 0 0"/>
+      <mass value="1.3729096e+00"/>
       <inertia ixx="8.7002718e-03" ixy="-4.7576583e-05" ixz="1.1160499e-04"
-        iyy="8.6195418e-03" iyz="-3.5422299e-06"
-        izz="1.4612727e-02" />
+               iyy="8.6195418e-03" iyz="-3.5422299e-06"
+               izz="1.4612727e-02" />
     </inertial>
   </link>
   <joint name="wheel_left_joint" type="continuous">
-    <parent link="base_link" />
-    <child link="wheel_left_link" />
-    <origin xyz="0.0 0.144 0.023" rpy="-1.57 0 0" />
-    <axis xyz="0 0 1" />
+    <parent link="base_link"/>
+    <child link="wheel_left_link"/>
+    <origin xyz="0.0 0.144 0.023" rpy="-1.57 0 0"/>
+    <axis xyz="0 0 1"/>
   </joint>
   <link name="wheel_left_link">
     <visual>
-      <origin xyz="0 0 0" rpy="1.57 0 0" />
-      <geometry>
-        <mesh filename="package://sim_env/meshes/turtlebot3/wheels/left_tire.stl" scale="0.001 0.001 0.001" />
-      </geometry>
-      <material name="dark" />
-    </visual>
-    <collision>
-      <origin xyz="0 0 0" rpy="0 0 0" />
-      <geometry>
-        <cylinder length="0.018" radius="0.033" />
+      <origin xyz="0 0 0" rpy="1.57 0 0"/>
+      <geometry>
+        <mesh filename="package://sim_env/meshes/turtlebot3/wheels/left_tire.stl" scale="0.001 0.001 0.001"/>
+      </geometry>
+      <material name="dark"/>
+    </visual>
+    <collision>
+      <origin xyz="0 0 0" rpy="0 0 0"/>
+      <geometry>
+        <cylinder length="0.018" radius="0.033"/>
       </geometry>
     </collision>
@@ -57,26 +57,26 @@
       <mass value="2.8498940e-02" />
       <inertia ixx="1.1175580e-05" ixy="-4.2369783e-11" ixz="-5.9381719e-09"
-        iyy="1.1192413e-05" iyz="-1.4400107e-11"
-        izz="2.0712558e-05" />
-    </inertial>
+               iyy="1.1192413e-05" iyz="-1.4400107e-11"
+               izz="2.0712558e-05" />
+      </inertial>
   </link>
   <joint name="wheel_right_joint" type="continuous">
-    <parent link="base_link" />
-    <child link="wheel_right_link" />
-    <origin xyz="0.0 -0.144 0.023" rpy="-1.57 0 0" />
-    <axis xyz="0 0 1" />
+    <parent link="base_link"/>
+    <child link="wheel_right_link"/>
+    <origin xyz="0.0 -0.144 0.023" rpy="-1.57 0 0"/>
+    <axis xyz="0 0 1"/>
   </joint>
   <link name="wheel_right_link">
     <visual>
-      <origin xyz="0 0 0" rpy="1.57 0 0" />
-      <geometry>
-        <mesh filename="package://sim_env/meshes/turtlebot3/wheels/right_tire.stl" scale="0.001 0.001 0.001" />
-      </geometry>
-      <material name="dark" />
-    </visual>
-    <collision>
-      <origin xyz="0 0 0" rpy="0 0 0" />
-      <geometry>
-        <cylinder length="0.018" radius="0.033" />
+      <origin xyz="0 0 0" rpy="1.57 0 0"/>
+      <geometry>
+        <mesh filename="package://sim_env/meshes/turtlebot3/wheels/right_tire.stl" scale="0.001 0.001 0.001"/>
+      </geometry>
+      <material name="dark"/>
+    </visual>
+    <collision>
+      <origin xyz="0 0 0" rpy="0 0 0"/>
+      <geometry>
+        <cylinder length="0.018" radius="0.033"/>
       </geometry>
     </collision>
@@ -85,18 +85,18 @@
       <mass value="2.8498940e-02" />
       <inertia ixx="1.1175580e-05" ixy="-4.2369783e-11" ixz="-5.9381719e-09"
-        iyy="1.1192413e-05" iyz="-1.4400107e-11"
-        izz="2.0712558e-05" />
-    </inertial>
+               iyy="1.1192413e-05" iyz="-1.4400107e-11"
+               izz="2.0712558e-05" />
+      </inertial>
   </link>
   <joint name="caster_back_right_joint" type="fixed">
-    <parent link="base_link" />
-    <child link="caster_back_right_link" />
-    <origin xyz="-0.177 -0.064 -0.004" rpy="-1.57 0 0" />
+    <parent link="base_link"/>
+    <child link="caster_back_right_link"/>
+    <origin xyz="-0.177 -0.064 -0.004" rpy="-1.57 0 0"/>
   </joint>
   <link name="caster_back_right_link">
     <collision>
-      <origin xyz="0 0.001 0" rpy="0 0 0" />
-      <geometry>
-        <box size="0.030 0.009 0.020" />
+      <origin xyz="0 0.001 0" rpy="0 0 0"/>
+      <geometry>
+        <box size="0.030 0.009 0.020"/>
       </geometry>
     </collision>
@@ -105,18 +105,18 @@
       <mass value="0.005" />
       <inertia ixx="0.001" ixy="0.0" ixz="0.0"
-        iyy="0.001" iyz="0.0"
-        izz="0.001" />
+               iyy="0.001" iyz="0.0"
+               izz="0.001" />
     </inertial>
   </link>
   <joint name="caster_back_left_joint" type="fixed">
-    <parent link="base_link" />
-    <child link="caster_back_left_link" />
-    <origin xyz="-0.177 0.064 -0.004" rpy="-1.57 0 0" />
+    <parent link="base_link"/>
+    <child link="caster_back_left_link"/>
+    <origin xyz="-0.177 0.064 -0.004" rpy="-1.57 0 0"/>
   </joint>
   <link name="caster_back_left_link">
     <collision>
-      <origin xyz="0 0.001 0" rpy="0 0 0" />
-      <geometry>
-        <box size="0.030 0.009 0.020" />
+      <origin xyz="0 0.001 0" rpy="0 0 0"/>
+      <geometry>
+        <box size="0.030 0.009 0.020"/>
       </geometry>
     </collision>
@@ -125,31 +125,31 @@
       <mass value="0.005" />
       <inertia ixx="0.001" ixy="0.0" ixz="0.0"
-        iyy="0.001" iyz="0.0"
-        izz="0.001" />
+               iyy="0.001" iyz="0.0"
+               izz="0.001" />
     </inertial>
   </link>
   <joint name="imu_joint" type="fixed">
-    <parent link="base_link" />
-    <child link="imu_link" />
-    <origin xyz="0.0 0 0.068" rpy="0 0 0" />
-  </joint>
-  <link name="imu_link" />
+    <parent link="base_link"/>
+    <child link="imu_link"/>
+    <origin xyz="0.0 0 0.068" rpy="0 0 0"/>
+  </joint>
+  <link name="imu_link"/>
   <joint name="scan_joint" type="fixed">
-    <parent link="base_link" />
-    <child link="base_scan" />
-    <origin xyz="-0.064 0 0.122" rpy="0 0 0" />
+    <parent link="base_link"/>
+    <child link="base_scan"/>
+    <origin xyz="-0.064 0 0.122" rpy="0 0 0"/>
   </joint>
   <link name="base_scan">
     <visual>
-      <origin xyz="0 0 0" rpy="0 0 0" />
-      <geometry>
-        <mesh filename="package://sim_env/meshes/turtlebot3/sensors/lds.stl" scale="0.001 0.001 0.001" />
-      </geometry>
-      <material name="dark" />
-    </visual>
-    <collision>
-      <origin xyz="0.015 0 -0.0065" rpy="0 0 0" />
-      <geometry>
-        <cylinder length="0.0315" radius="0.055" />
+      <origin xyz="0 0 0" rpy="0 0 0"/>
+      <geometry>
+        <mesh filename="package://sim_env/meshes/turtlebot3/sensors/lds.stl" scale="0.001 0.001 0.001"/>
+      </geometry>
+      <material name="dark"/>
+    </visual>
+    <collision>
+      <origin xyz="0.015 0 -0.0065" rpy="0 0 0"/>
+      <geometry>
+        <cylinder length="0.0315" radius="0.055"/>
       </geometry>
     </collision>
@@ -158,28 +158,28 @@
       <origin xyz="0 0 0" />
       <inertia ixx="0.001" ixy="0.0" ixz="0.0"
-        iyy="0.001" iyz="0.0"
-        izz="0.001" />
+               iyy="0.001" iyz="0.0"
+               izz="0.001" />
     </inertial>
   </link>
   <joint name="camera_joint" type="fixed">
-    <origin xyz="0.064 -0.065 0.094" rpy="0 0 0" />
-    <parent link="base_link" />
-    <child link="camera_link" />
+    <origin xyz="0.064 -0.065 0.094" rpy="0 0 0"/>
+    <parent link="base_link"/>
+    <child link="camera_link"/>
   </joint>
   <link name="camera_link">
     <visual>
-      <origin xyz="0 0 0" rpy="1.57 0 1.57" />
-      <geometry>
-        <mesh filename="package://sim_env/meshes/turtlebot3/sensors/r200.dae" />
-      </geometry>
-    </visual>
-    <collision>
-      <origin xyz="0.003 0.065 0.007" rpy="0 0 0" />
-      <geometry>
-        <box size="0.012 0.132 0.020" />
+     <origin xyz="0 0 0" rpy="1.57 0 1.57"/>
+      <geometry>
+       <mesh filename="package://sim_env/meshes/turtlebot3/sensors/r200.dae" />
+      </geometry>
+    </visual>
+    <collision>
+      <origin xyz="0.003 0.065 0.007" rpy="0 0 0"/>
+      <geometry>
+        <box size="0.012 0.132 0.020"/>
       </geometry>
     </collision>
     <!-- This inertial field needs doesn't contain reliable data!! -->
-    <!--   <inertial>
+<!--   <inertial>
       <mass value="0.564" />
       <origin xyz="0 0 0" />
@@ -190,26 +190,26 @@
   </link>
   <joint name="camera_rgb_joint" type="fixed">
-    <origin xyz="${r200_cam_rgb_px} ${r200_cam_rgb_py} ${r200_cam_rgb_pz}" rpy="0 0 0" />
-    <parent link="camera_link" />
-    <child link="camera_rgb_frame" />
-  </joint>
-  <link name="camera_rgb_frame" />
+    <origin xyz="${r200_cam_rgb_px} ${r200_cam_rgb_py} ${r200_cam_rgb_pz}" rpy="0 0 0"/>
+    <parent link="camera_link"/>
+    <child link="camera_rgb_frame"/>
+  </joint>
+  <link name="camera_rgb_frame"/>
   <joint name="camera_rgb_optical_joint" type="fixed">
-    <origin xyz="0 0 0" rpy="-1.57 0 -1.57" />
-    <parent link="camera_rgb_frame" />
-    <child link="camera_rgb_optical_frame" />
-  </joint>
-  <link name="camera_rgb_optical_frame" />
+    <origin xyz="0 0 0" rpy="-1.57 0 -1.57"/>
+    <parent link="camera_rgb_frame"/>
+    <child link="camera_rgb_optical_frame"/>
+  </joint>
+  <link name="camera_rgb_optical_frame"/>
   <joint name="camera_depth_joint" type="fixed">
-    <origin xyz="${r200_cam_rgb_px} ${r200_cam_rgb_py + r200_cam_depth_offset} ${r200_cam_rgb_pz}" rpy="0 0 0" />
-    <parent link="camera_link" />
-    <child link="camera_depth_frame" />
-  </joint>
-  <link name="camera_depth_frame" />
+    <origin xyz="${r200_cam_rgb_px} ${r200_cam_rgb_py + r200_cam_depth_offset} ${r200_cam_rgb_pz}" rpy="0 0 0"/>
+    <parent link="camera_link"/>
+    <child link="camera_depth_frame"/>
+  </joint>
+  <link name="camera_depth_frame"/>
   <joint name="camera_depth_optical_joint" type="fixed">
-    <origin xyz="0 0 0" rpy="-1.57 0 -1.57" />
-    <parent link="camera_depth_frame" />
-    <child link="camera_depth_optical_frame" />
-  </joint>
-  <link name="camera_depth_optical_frame" />
+    <origin xyz="0 0 0" rpy="-1.57 0 -1.57"/>
+    <parent link="camera_depth_frame"/>
+    <child link="camera_depth_optical_frame"/>
+  </joint>
+  <link name="camera_depth_optical_frame"/>
 </robot>

File: src/sim_env/urdf/turtlebot3_waffle/turtlebot3_waffle.xacro (robot description, xacro)
@@ -1,6 +1,6 @@
-<?xml version="1.0"?>
+<?xml version="1.0" ?>
 <robot name="turtlebot3_waffle" xmlns:xacro="http://ros.org/wiki/xacro">
-  <xacro:include filename="$(find sim_env)/urdf/turtlebot3_waffle/common_properties.xacro" />
-  <xacro:include filename="$(find sim_env)/urdf/turtlebot3_waffle/turtlebot3_waffle.gazebo.xacro" />
-  <xacro:include filename="$(find sim_env)/urdf/turtlebot3_waffle/turtlebot3_waffle.urdf.xacro" />
+  <xacro:include filename="$(find sim_env)/urdf/turtlebot3_waffle/common_properties.xacro"/>
+  <xacro:include filename="$(find sim_env)/urdf/turtlebot3_waffle/turtlebot3_waffle.gazebo.xacro"/>
+  <xacro:include filename="$(find sim_env)/urdf/turtlebot3_waffle/turtlebot3_waffle.urdf.xacro"/>
 </robot>

File: src/sim_env/urdf/turtlebot3_waffle_pi/common_properties.xacro (robot description, xacro)
@@ -1,34 +1,34 @@
-<?xml version="1.0"?>
+<?xml version="1.0" ?>
 <robot name="xacro_properties" xmlns:xacro="http://ros.org/wiki/xacro">
   <!-- Init colour -->
   <material name="black">
-    <color rgba="0.0 0.0 0.0 1.0" />
+      <color rgba="0.0 0.0 0.0 1.0"/>
   </material>
   <material name="dark">
-    <color rgba="0.3 0.3 0.3 1.0" />
+    <color rgba="0.3 0.3 0.3 1.0"/>
   </material>
   <material name="light_black">
-    <color rgba="0.4 0.4 0.4 1.0" />
+    <color rgba="0.4 0.4 0.4 1.0"/>
   </material>
   <material name="blue">
-    <color rgba="0.0 0.0 0.8 1.0" />
+    <color rgba="0.0 0.0 0.8 1.0"/>
   </material>
   <material name="green">
-    <color rgba="0.0 0.8 0.0 1.0" />
+    <color rgba="0.0 0.8 0.0 1.0"/>
   </material>
   <material name="grey">
-    <color rgba="0.5 0.5 0.5 1.0" />
+    <color rgba="0.5 0.5 0.5 1.0"/>
   </material>
   <material name="orange">
-    <color rgba="${255/255} ${108/255} ${10/255} 1.0" />
+    <color rgba="${255/255} ${108/255} ${10/255} 1.0"/>
   </material>
   <material name="brown">
-    <color rgba="${222/255} ${207/255} ${195/255} 1.0" />
+    <color rgba="${222/255} ${207/255} ${195/255} 1.0"/>
   </material>
   <material name="red">
-    <color rgba="0.8 0.0 0.0 1.0" />
+    <color rgba="0.8 0.0 0.0 1.0"/>
   </material>
   <material name="white">
-    <color rgba="1.0 1.0 1.0 1.0" />
+    <color rgba="1.0 1.0 1.0 1.0"/>
   </material>
 </robot>

File: src/sim_env/urdf/turtlebot3_waffle_pi/turtlebot3_waffle_pi.gazebo.xacro (robot description, xacro)
@@ -1,7 +1,7 @@
 <?xml version="1.0"?>
 <robot name="turtlebot3_waffle_pi_sim" xmlns:xacro="http://ros.org/wiki/xacro">
-  <xacro:arg name="laser_visual" default="false" />
-  <xacro:arg name="camera_visual" default="false" />
-  <xacro:arg name="imu_visual" default="false" />
+  <xacro:arg name="laser_visual"  default="false"/>
+  <xacro:arg name="camera_visual" default="false"/>
+  <xacro:arg name="imu_visual"    default="false"/>
   <gazebo reference="base_link">
     <material>Gazebo/DarkGrey</material>
@@ -134,4 +134,5 @@
     </sensor>
   </gazebo>
+<!--link : https://www.raspberrypi.org/documentation/hardware/camera/-->
   <gazebo reference="camera_rgb_frame">
     <sensor type="camera" name="Pi Camera">
@@ -139,14 +140,14 @@
       <visualize>$(arg camera_visual)</visualize>
       <camera>
-        <horizontal_fov>1.085595</horizontal_fov>
-        <image>
-          <width>640</width>
-          <height>480</height>
-          <format>R8G8B8</format>
-        </image>
-        <clip>
-          <near>0.03</near>
-          <far>100</far>
-        </clip>
+          <horizontal_fov>1.085595</horizontal_fov>
+          <image>
+              <width>640</width>
+              <height>480</height>
+              <format>R8G8B8</format>
+          </image>
+          <clip>
+              <near>0.03</near>
+              <far>100</far>
+          </clip>
       </camera>
       <plugin name="camera_controller" filename="libgazebo_ros_camera.so">
